File: Byggern_Schematics/Byggern_Schematics.kicad_sch (KiCad schematic)
At the start: 21 parts, among them IC1 MAX233, IC2 SN74ALS573CN, IC3 7164S25YG, IC4 SN74HC00N, J1 Conn_02x05_Odd_Even, J2 DE9_Socket, J3 V_{In} Plug, J4 GND Plug, SW1 Reset, U1 ATmega162-16P, U2 LM7805_TO220, Y1 4.9152MHz

Commit message: schematics ting
Parts:
- added IC5: MAX156BCNG+, Samacsys:DIP794W56P254L3054H457Q24N, symbol Samacsys:MAX156BCNG+
Connections:
- net +5V: no longer IC3.28 (VCC)
- net GND: no longer IC2.1 (~{OE}), IC3.14 (GND)
- net ~{RD}: no longer names the net of IC3.22 (~{OE})
- net ~{WE}: no longer names the net of IC3.27 (~{WE})
Other:
- added sheet AVR ATmega162 (ATmega162.kicad_sch)
- added sheet Digital Interface (Digital_Interface.kicad_sch)
- added sheet Ekstern minne (ekstern_minne.kicad_sch)

Commit message: Byggern sjematikk for ADC done
Parts:
- removed C5: 1u, symbol Device:C
- removed IC1: MAX233, Samacsys:DIP762W56P254L2616H457Q20N, symbol Samacsys:MAX233CPP+G36
- removed IC2: SN74ALS573CN, Samacsys:DIP794W53P254L2540H508Q20N, symbol Samacsys:SN74ALS573CN
- removed IC3: 7164S25YG, Samacsys:7164S25YG, symbol Samacsys:7164S25YG
- removed IC4: SN74HC00N, Samacsys:DIP794W53P254L1930H508Q14N, symbol Samacsys:SN74HC00N
- removed IC5: MAX156BCNG+, Samacsys:DIP794W56P254L3054H457Q24N, symbol Samacsys:MAX156BCNG+
- removed J1: Conn_02x05_Odd_Even, symbol Connector_Generic:Conn_02x05_Odd_Even
- removed J2: DE9_Socket, symbol Connector:DE9_Socket
- added C8: 100n, symbol Device:C
- added J6: IO_Board, Connector_IDC:IDC-Header_2x07_P2.54mm_Vertical, symbol Connector_Generic:Conn_02x07_Counter_Clockwise
- added R3: 33R, symbol Device:R
Connections:
- net  ~{RESET} is gone; now on net ~{RESET}: C1.2, R1.2, U1.9 (~{RESET})
- net +5V: now also J6.1 (Pin_1)
- net ALE: now also C8.2, R3.1; no longer U1.30 (PE1)
- net GND: now also C8.1, J6.2 (Pin_2)
- net PD2: now reaches U1.12 (PD2)
- net CLK: now reaches U1.14 (PD4)
- net PC0: now reaches U1.21 (PC0)
- net PC1: now reaches U1.22 (PC1)
- net PC2: now reaches U1.23 (PC2)
- net PC3: now reaches U1.24 (PC3)
- net PA7: now reaches U1.32 (PA7)
- net PA6: now reaches U1.33 (PA6)
- net PA5: now reaches U1.34 (PA5)
- net PA4: now reaches U1.35 (PA4)
- net PA3: now reaches U1.36 (PA3)
- net PA2: now reaches U1.37 (PA2)
- net PA1: now reaches U1.38 (PA1)
- net PA0: now reaches U1.39 (PA0)
- net RD renamed ~{RD}
- net WR renamed ~{WR}
- new net BTN: J6.3 (Pin_3)
- new net DISPLAY_D/~{C}: J6.14 (Pin_14)
- new net DISPLAY_~{CS}: J6.13 (Pin_13)
- new net DISPLAY_~{RES}: J6.8 (Pin_8)
- new net IO_~{CS}: J6.12 (Pin_12)
- new net JOYSTICK_X: J6.7 (Pin_7)
- new net JOYSTICK_Y: J6.6 (Pin_6)
- new net MISO: J6.10 (Pin_10)
- new net MOSI: J6.11 (Pin_11)
- new net PE1: R3.2, U1.30 (PE1)
- new net SCK: J6.9 (Pin_9)
- new net TOUCH_X: J6.5 (Pin_5)
- new net TOUCH_Y: J6.4 (Pin_4)
- no-connect marks 15 -> 11
Other:
- removed sheet AVR ATmega162
- sheet Digital Interface ports: added JTAG_TCK, JTAG_TDI, JTAG_TDO, JTAG_TMS, UART_RX, UART_TX; removed none
- sheet Ekstern minne ports: added AIN0, AIN1, AIN2, AIN3, ALE, CLK, PA, PC, ~{BUSY}, ~{RD}, ~{WR}; removed none

Commit message: Schematic udated
Connections:
- net DISPLAY_~{RES} is gone; now on net ~{RESET}: J6.8 (Pin_8)
- net +5V: now also J6.2 (Pin_2); no longer J6.1 (Pin_1)
- net ALE: now also C8.1, R3.2; no longer C8.2, R3.1
- net BTN: now also U1.1 (PB0)
- net DISPLAY_D/~{C}: now also U1.3 (PB2)
- net DISPLAY_~{CS}: now also U1.4 (PB3)
- net GND: now also C8.2, J6.1 (Pin_1); no longer C8.1, J6.2 (Pin_2)
- net IO_~{CS}: now also U1.5 (PB4)
- net MISO: now also U1.7 (PB6)
- net MOSI: now also U1.6 (PB5)
- net PE1: now also R3.1; no longer R3.2
- net SCK: now also U1.8 (PB7)
- net ~{BUSY}: now reaches U1.13 (PD3)
- net CAN_~{CS}: now reaches U1.2 (PB1)
- net JOYSTICK_X renamed Ekstern minne/AIN0
- net JOYSTICK_Y renamed Ekstern minne/AIN1
- net PD2 renamed ~{INT}
- net TOUCH_X renamed Ekstern minne/AIN2
- net TOUCH_Y renamed Ekstern minne/AIN3
- no-connect marks 11 -> 3
Other:
- sheet Digital Interface ports: added MISO, MOSI, SCK, ~{CS}, ~{INT}, ~{RESET}; removed none
- sheet Ekstern minne ports: added CTRL; removed ALE, CLK, ~{BUSY}, ~{RD}, ~{WR}
- moved on the sheet: U1

Commit message: Finnished schematic
Parts:
- removed C1: 100n, symbol Device:C
- added C4: 100n, symbol Device:C
- renumbered C6 to C1, C3 to C2, C7 to C3, C2 to C5, C4 to C6, C8 to C7, J3 to J1, J4 to J2, J6 to J3, R2 to R1, R1 to R2, U2 to U1, U1 to U2
Connections:
- net GND: now also C4.2
- net ~{RESET}: now also C4.1
- net BTN renamed JOY_BTN
- net Ekstern minne/AIN0 renamed JOYSTICK_X
- net Ekstern minne/AIN1 renamed JOYSTICK_Y
- net Ekstern minne/AIN2 renamed TOUCH_X
- net Ekstern minne/AIN3 renamed TOUCH_Y
- net RXD0 renamed RX
- net SCK renamed PB7
- net TXD0 renamed TX
Other:
- note added: "ADC"
- note added: "ALE Lowpass filter"
- note added: "CAN"
- note added: "Crystall oscillator"
- note added: "IO-Board Connector"
- note added: "JTAG"
- note added: "Paralell interface peripherals"
- note added: "Power circuitry"
- note added: "RS232"
- note added: "Reset circuitry"
- note added: "SRAM"
- note added: "Serial interface peripherals"
- company: (none) -> Gruppe 31
- title: Peneste shittet ever -> Veldig pent yup yup
- moved on the sheet: C1, C2, C3, C5, C6, C7, J1, J2, J3, R1, R2, R3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

Commit message: Liten Schematic endring
Parts:
- renumbered C4 to C1, C6 to C2, C2 to C3, C5 to C4, C1 to C5, C3 to C6, J3 to J1, J1 to J2, J2 to J3, U2 to U1, U1 to U2

Commit message: Schematic endring
Other:
- note added: "Note that grey signals on the schematic are white IRL"
Changed lines of the file:
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@@
+		)
+	)
+	(text "Note that grey signals on the schematic are white IRL"
+		(exclude_from_sim no)
+		(at 253.238 46.228 0)
+		(effects
+			(font
+				(size 1.27 1.27)
+			)
 		)
 	)

Commit message: Små endringer til schematic
Parts:
- removed C1, C2, C7: 100n, symbol Device:C
- removed C3, C4: 22p, symbol Device:C
- removed C5: 1u, symbol Device:C
- removed C6: 10u, symbol Device:C_Polarized
- removed J1: IO_Board, Connector_IDC:IDC-Header_2x07_P2.54mm_Vertical, symbol Connector_Generic:Conn_02x07_Counter_Clockwise
- removed J2: V_{In} Plug, symbol Connector:Conn_01x01_Socket
- removed J3: GND Plug, symbol Connector:Conn_01x01_Socket
- removed R1: 10k, symbol Device:R
- removed R2: 330R, symbol Device:R
- removed R3: 33R, symbol Device:R
- removed SW1: Reset, symbol Switch:SW_Push
- removed U1: ATmega162-16P, Package_DIP:DIP-40_W15.24mm, symbol MCU_Microchip_ATmega:ATmega162-16P
- removed U2: LM7805_TO220, Package_TO_SOT_THT:TO-220-3_Vertical, symbol Regulator_Linear:LM7805_TO220
- removed Y1: 4.9152MHz, symbol Device:Crystal
Connections:
- no-connect marks 3 -> 0
Other:
- removed sheet Digital Interface
- removed sheet Ekstern minne
- added sheet Node 1 (Node1.kicad_sch)
- added sheet Node 2 (Node2.kicad_sch)
- added sheet Ping Pong Interface (ping_pong_board.kicad_sch)
- note removed: "ADC"
- note removed: "ALE Lowpass filter"
- note removed: "CAN"
- note removed: "Crystall oscillator"
- note removed: "IO-Board Connector"
- note removed: "JTAG"
- note removed: "Note that grey signals on the schematic are white IRL"
- note removed: "Paralell interface peripherals"
- note removed: "Power circuitry"
- note removed: "RS232"
- note removed: "Reset circuitry"
- note removed: "SRAM"
- note removed: "Serial interface peripherals"
