File: Byggern_Schematics/Byggern_Schematics.kicad_sch (KiCad schematic)
At the start: 0 parts

Commit message: A lot of schematic changes
Parts:
- added A1: Arduino Duo, Module:Arduino_UNO_R3, symbol MCU_Module:Arduino_UNO_R3
- added A2: Motor Shield, Module:Arduino_UNO_R3, symbol MCU_Module:Arduino_UNO_R3
- added C1, C2, C56, C59, C60: 100n, symbol Device:C
- added C54: 1u, symbol Device:C
- added C55, C58: 22p, symbol Device:C
- added C57: 10u, symbol Device:C_Polarized
- added D1: IR Emitter, LED_THT:LED_D3.0mm_IRBlack, symbol LED:TSAL4400
- added D2: Photodiode, symbol Device:D_Photo
- added D4: Snubber, Diode_THT:D_DO-41_SOD81_P10.16mm_Horizontal, symbol Diode:1N4005
- added J1, J3: Conn_01x05_Pin, symbol Connector:Conn_01x05_Pin
- added J18: IO_Board, Connector_IDC:IDC-Header_2x07_P2.54mm_Vertical, symbol Connector_Generic:Conn_02x07_Counter_Clockwise
- added J2, J4: Conn_01x05_Socket, symbol Connector:Conn_01x05_Socket
- added J5: Conn_01x06_Pin, symbol Connector:Conn_01x06_Pin
- added J6: Conn_01x06_Socket, symbol Connector:Conn_01x06_Socket
- added K1: G5V-2, Relay_THT:Relay_DPDT_Omron_G5V-2, symbol Relay:G5V-2
- added L1: Solenoide, symbol Device:L
- added M1: Motor_Servo, symbol Motor:Motor_Servo
- added M2: Motor_DC, symbol Motor:Motor_DC
- added Q2: MPSA56, Package_TO_SOT_THT:TO-92_Inline, symbol Transistor_BJT:MPSA92
- added R1, R3: 47R, symbol Device:R
- added R13: 10k, symbol Device:R
- added R14, R4: 330R, symbol Device:R
- added R15: 33R, symbol Device:R
- added R2: 1M, symbol Device:R
- added R5: 1k, symbol Device:R
- added SW1: RotaryEncoder, symbol Device:RotaryEncoder
- added SW3: Reset, symbol Switch:SW_Push
- added U1: MCP602, symbol Amplifier_Operational:MCP602
- added U11: LM7805_TO220, Package_TO_SOT_THT:TO-220-3_Vertical, symbol Regulator_Linear:LM7805_TO220
- added U12: ATmega162-16P, Package_DIP:DIP-40_W15.24mm, symbol MCU_Microchip_ATmega:ATmega162-16P
- added V1, V3: 1, symbol Simulation_SPICE:VDC
- added Y6: 4.9152MHz, symbol Device:Crystal
Connections:
- new net: C1.2, R2.2, U1.1, U1.5 (+)
- new net: C1.1, J4.9 (Pin_4), R2.1, U1.2 (-)
- new net: J2.5 (Pin_5), K1.1
- new net: D4.1 (K), K1.4, Q2.3 (C)
- new net: R4.2, R5.1, U1.6 (-)
- new net: R5.2, U1.7
- new net: Q2.2 (B), R3.2
- new net: A1. (CANTX0), A2. (Servo_GND) (x2)
- new net: A1.20 (D20/SDA), A2. (Servo_GND)
- new net: A1.21 (D21/SCL), A2. (Servo_GND)
- new net: A1.4 (D4), A2. (Servo_GND)
- new net: A1.5 (D5), A2. (Servo_GND)
- new net: A1.7 (D7), A2. (Servo_GND)
- new net: D1.1 (K), J3.10 (Pin_5)
- new net: J3.6 (Pin_1), M1.1 (PWM)
- new net: J3.7 (Pin_2), M1.2 (+)
- new net: J3.8 (Pin_3), M1.3 (-)
- new net: D2.1 (K), J3.9 (Pin_4)
- new net: J1.5 (Pin_5), L1.1
- new net: J1.4 (Pin_4), L1.2
- new net: J4.10 (Pin_5), R1.1
- new net: A2. (Servo_GND), J4.6 (Pin_1)
- new net: A2. (Servo_GND), J4.7 (Pin_2)
- new net: A2. (Servo_GND), J4.8 (Pin_3)
- new net: D2.2 (A), J1.2 (Pin_2)
- new net: D1.2 (A), J1.1 (Pin_1)
- new net +12V: K1.3
- new net +3V3: A1. (CANTX0), C2.2, J2.1 (Pin_1), Q2.1 (E), U1.8 (V+)
- new net +5V: C57.1, C59.1, J18.2 (Pin_2), R13.2, U11.3 (VO), U12.40 (VCC)
- new net +V_{IN}: C54.2, U11.1 (VI), V1.1, V3.1
- new net ALE: C60.1, R15.2
- new net CANH: A2. (Servo_GND)
- new net CANL: A2. (Servo_GND)
- new net CAN_~{CS}: U12.2 (PB1)
- new net CLK: U12.14 (PD4)
- new net DISPLAY_D/~{C}: J18.14 (Pin_14), U12.3 (PB2)
- new net DISPLAY_~{CS}: J18.13 (Pin_13), U12.4 (PB3)
- new net Encoder_3V3: A2. (Servo_GND)
- new net Encoder_GND: A2. (Servo_GND)
- new net GND: A1. (CANTX0), C2.1, C54.1, C55.1, C56.2, C57.2, C58.1, C59.2, C60.2, D4.2 (A), J18.1 (Pin_1), J2.2 (Pin_2), J2.4 (Pin_4), K1.5, R1.2, R4.1, SW3.1, U1.3 (+), U1.4 (V-), U11.2 (GND), U12.20 (GND), V1.2, V3.2
- new net IO_~{CS}: J18.12 (Pin_12), U12.5 (PB4)
- new net JOYSTICK_X: J18.7 (Pin_7)
- new net JOYSTICK_Y: J18.6 (Pin_6)
- new net JOY_BTN: J18.3 (Pin_3), U12.1 (PB0)
- new net JTAG_TCK: U12.25 (PC4)
- new net JTAG_TDI: U12.28 (PC7)
- new net JTAG_TDO: U12.27 (PC6)
- new net JTAG_TMS: U12.26 (PC5)
- new net MISO: J18.10 (Pin_10), U12.7 (PB6)
- new net MOSI: J18.11 (Pin_11), U12.6 (PB5)
- new net PA0: U12.39 (PA0)
- new net PA1: U12.38 (PA1)
- new net PA2: U12.37 (PA2)
- new net PA3: U12.36 (PA3)
- new net PA4: U12.35 (PA4)
- new net PA5: U12.34 (PA5)
- new net PA6: U12.33 (PA6)
- new net PA7: U12.32 (PA7)
- new net PB7: J18.9 (Pin_9), U12.8 (PB7)
- new net PC0: U12.21 (PC0)
- new net PC1: U12.22 (PC1)
- new net PC2: U12.23 (PC2)
- new net PC3: U12.24 (PC3)
- new net PE1: R15.1, U12.30 (PE1)
- new net QUAD_A: A2. (Servo_GND)
- new net QUAD_B: A2. (Servo_GND)
- new net RX: U12.10 (PD0)
- new net TOUCH_X: J18.5 (Pin_5)
- new net TOUCH_Y: J18.4 (Pin_4)
- new net TX: U12.11 (PD1)
- new net XTAL1: C55.2, U12.19 (XTAL1), Y6.2
- new net XTAL2: C58.2, U12.18 (XTAL2), Y6.1
- new net ~{BUSY}: U12.13 (PD3)
- new net ~{INT}: U12.12 (PD2)
- new net ~{RD}: U12.17 (PD7)
- new net ~{RESET_SW}: R13.1, R14.1, SW3.2
- new net ~{RESET}: C56.1, J18.8 (Pin_8), R14.2, U12.9 (~{RESET})
- new net ~{WR}: U12.16 (PD6)
- no-connect marks 0 -> 25
Other:
- removed sheet Node 1
- removed sheet Node 2
- removed sheet Ping Pong Interface
- added sheet Digital Interface (Digital_Interface.kicad_sch)
- added sheet Ekstern minne (ekstern_minne.kicad_sch)
- note added: "ADC"
- note added: "ALE Lowpass filter"
- note added: "CAN"
- note added: "Crystall oscillator"
- note added: "IO-Board Connector"
- note added: "JTAG"
- note added: "Note that grey signals on the schematic are white IRL"
- note added: "Paralell interface peripherals"
- note added: "Power circuitry"
- note added: "RS232"
- note added: "Reset circuitry"
- note added: "SRAM"
- note added: "Serial interface peripherals"

Commit message: Fjærna write protection
Parts:
- removed J5: Conn_01x06_Pin, symbol Connector:Conn_01x06_Pin
- removed J6: Conn_01x06_Socket, symbol Connector:Conn_01x06_Socket
- added R6: 100k, symbol Device:R
- R3: value 47R -> 1k
Connections:
- net +3V3: now also J4.10 (Pin_5); no longer J2.1 (Pin_1)
- net Encoder_3V3: now also SW1.VCC
- net Encoder_GND: now also SW1.GND (VCC)
- net GND: now also R6.1
- net QUAD_A: now also SW1.A
- net QUAD_B: now also SW1.B
- net at R5.2, U1.7: now also A1. (CANTX0)
- net at J3.10 (Pin_5): now also D1.2 (A); no longer D1.1 (K)
- net at R3.1: now also A1. (CANTX0), R6.2
- net at M2.1 (+): now also A2. (Servo_GND)
- net at M2.2 (-): now also A2. (Servo_GND)
- net at R1.1: now also J2.1 (Pin_1); no longer J4.10 (Pin_5)
- net at J1.1 (Pin_1): now also D1.1 (K); no longer D1.2 (A)
- new net: A1. (CANTX0), A2. (Servo_GND) (x2)
Other:
- moved on the sheet: C54, C55, C56, C57, C58, C59, C60, J18, R13, R14, R15, SW3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

Commit message: Små schematic endringer
Parts:
- removed V1: 1, symbol Simulation_SPICE:VDC
- added V4: 1, symbol Simulation_SPICE:VDC
Connections:
- net +V_{IN}: now also A2. (Servo_GND)
- net GND: now also A2. (Servo_GND); no longer J2.4 (Pin_4)
- net at K1.1: no longer J2.5 (Pin_5)
- net at K1.6: now also V4.1
- net at K1.8: now also J2.5 (Pin_5)
- net +12V: no longer names the net of K1.3
- new net: A1. (CANTX0), A2. (Servo_GND) (x2)
- new net: J2.4 (Pin_4), V4.2
Other:
- moved on the sheet: D4, K1, Q2, R3, R6, V3

Commit message: Små schematic endringer og eksporterte som PDF
Connections:
- new net: A1. (CANTX0), A2. (Servo_GND) (x2)
Other:
- note added: "Arduino with shield"
- note added: "Little breadboard"
- note added: "Motorbrett"
- note added: "NODE 1"
- note added: "NODE 2"
Changed lines of the file:
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@@
 		)
 	)
+	(text "NODE 2"
+		(exclude_from_sim no)
+		(at 304.038 25.654 0)
+		(effects
+			(font
+				(size 5.08 5.08)
+				(thickness 1.016)
+				(bold yes)
+			)
+		)
+	)
+	(text "Motorbrett"
+		(exclude_from_sim no)
+		(at 355.6 189.23 0)
+		(effects
+			(font
+				(size 2.54 2.54)
+				(thickness 1.016)
+				(bold yes)
+			)
+		)
+	)
 	(text "ALE Lowpass filter"
 		(exclude_from_sim no)
@@
 		)
 	)
+	(text "NODE 1"
+		(exclude_from_sim no)
+		(at 117.856 28.448 0)
+		(effects
+			(font
+				(size 5.08 5.08)
+				(thickness 1.016)
+				(bold yes)
+			)
+		)
+	)
 	(text "Note that grey signals on the schematic are white IRL"
 		(exclude_from_sim no)
-		(at 251.46 40.64 0)
+		(at 196.85 44.45 0)
 		(effects
 			(font
@@
 		)
 	)
+	(text "Arduino with shield"
+		(exclude_from_sim no)
+		(at 288.798 120.396 0)
+		(effects
+			(font
+				(size 2.54 2.54)
+				(thickness 1.016)
+				(bold yes)
+			)
+		)
+	)
 	(text "JTAG"
 		(exclude_from_sim no)
@@
 		)
 	)
+	(text "Little breadboard"
+		(exclude_from_sim no)
+		(at 265.43 213.868 0)
+		(effects
+			(font
+				(size 2.54 2.54)
+				(thickness 1.016)
+				(bold yes)
+			)
+		)
+	)
 	(text "Serial interface peripherals"
 		(exclude_from_sim no)
@@
 			(table_cell "Color"
 				(exclude_from_sim no)
-				(at 235.077 15.367 0)
+				(at 180.467 19.177 0)
 				(size 10.16 2.54)
 				(margins 0.9525 0.9525 0.9525 0.9525)
@@
 			(table_cell "Type"
 				(exclude_from_sim no)
-				(at 245.237 15.367 0)
+				(at 190.627 19.177 0)
 				(size 22.86 2.54)
 				(margins 0.9525 0.9525 0.9525 0.9525)
@@
 			(table_cell "Red"
 				(exclude_from_sim no)
-				(at 235.077 17.907 0)
+				(at 180.467 21.717 0)
 				(size 10.16 2.54)
 				(margins 0.9525 0.9525 0.9525 0.9525)
@@
 			(table_cell "5V"
 				(exclude_from_sim no)
-				(at 245.237 17.907 0)
+				(at 190.627 21.717 0)
 				(size 22.86 2.54)
 				(margins 0.9525 0.9525 0.9525 0.9525)
@@
 			(table_cell "Orange"
 				(exclude_from_sim no)
-				(at 235.077 20.447 0)
+				(at 180.467 24.257 0)
 				(size 10.16 2.54)
 				(margins 0.9525 0.9525 0.9525 0.9525)
@@
 			(table_cell "Power that isn't GND"
 				(exclude_from_sim no)
-				(at 245.237 20.447 0)
+				(at 190.627 24.257 0)
 				(size 22.86 2.54)
 				(margins 0.9525 0.9525 0.9525 0.9525)
@@
 			(table_cell "Black"
 				(exclude_from_sim no)
-				(at 235.077 22.987 0)
+				(at 180.467 26.797 0)
 				(size 10.16 2.54)
 				(margins 0.9525 0.9525 0.9525 0.9525)
@@
 			(table_cell "GND"
 				(exclude_from_sim no)
-				(at 245.237 22.987 0)
+				(at 190.627 26.797 0)
 				(size 22.86 2.54)
 				(margins 0.9525 0.9525 0.9525 0.9525)
@@
 			(table_cell "Brown"
 				(exclude_from_sim no)
-				(at 235.077 25.527 0)
+				(at 180.467 29.337 0)
 				(size 10.16 2.54)
 				(margins 0.9525 0.9525 0.9525 0.9525)
@@
 			(table_cell "Analog signal"
 				(exclude_from_sim no)
-				(at 245.237 25.527 0)
+				(at 190.627 29.337 0)
 				(size 22.86 2.54)
 				(margins 0.9525 0.9525 0.9525 0.9525)
@@
 			(table_cell "Blue"
 				(exclude_from_sim no)
-				(at 235.077 28.067 0)
+				(at 180.467 31.877 0)
 				(size 10.16 2.54)
 				(margins 0.9525 0.9525 0.9525 0.9525)
@@
 			(table_cell "Parallel bus signal"
 				(exclude_from_sim no)
-				(at 245.237 28.067 0)
+				(at 190.627 31.877 0)
 				(size 22.86 2.54)
 				(margins 0.9525 0.9525 0.9525 0.9525)
@@
 			(table_cell "Green"
 				(exclude_from_sim no)
-				(at 235.077 30.607 0)
+				(at 180.467 34.417 0)
 				(size 10.16 2.54)
 				(margins 0.9525 0.9525 0.9525 0.9525)
@@
 			(table_cell "Serial signals"
 				(exclude_from_sim no)
-				(at 245.237 30.607 0)
+				(at 190.627 34.417 0)
 				(size 22.86 2.54)
 				(margins 0.9525 0.9525 0.9525 0.9525)
@@
 			(table_cell "Yellow"
 				(exclude_from_sim no)
-				(at 235.077 33.147 0)
+				(at 180.467 36.957 0)
 				(size 10.16 2.54)
 				(margins 0.9525 0.9525 0.9525 0.9525)
@@
 			(table_cell "Digital signal"
 				(exclude_from_sim no)
-				(at 245.237 33.147 0)
+				(at 190.627 36.957 0)
 				(size 22.86 2.54)
 				(margins 0.9525 0.9525 0.9525 0.9525)
@@
 			(table_cell "Grey"
 				(exclude_from_sim no)
-				(at 235.077 35.687 0)
+				(at 180.467 39.497 0)
 				(size 10.16 2.54)
 				(margins 0.9525 0.9525 0.9525 0.9525)
@@
 			(table_cell "Control signal"
 				(exclude_from_sim no)
-				(at 245.237 35.687 0)
+				(at 190.627 39.497 0)
 				(size 22.86 2.54)
 				(margins 0.9525 0.9525 0.9525 0.9525)
