File: Byggern_Schematics/Digital_Interface.kicad_sch (KiCad schematic)
At the start: 0 parts

Commit message: Byggern sjematikk for ADC done
Parts:
- added C11: 1u, symbol Device:C
- added IC6: MAX233, Samacsys:DIP762W56P254L2616H457Q20N, symbol Samacsys:MAX233CPP+G36
- added J2: Conn_02x05_Odd_Even, symbol Connector_Generic:Conn_02x05_Odd_Even
- added J5: DE9_Socket, symbol Connector:DE9_Socket
Connections:
- new net +5V: C11.2, IC6.7 (VCC), J2.4 (Pin_4)
- new net C2+: IC6.11 (C2+), IC6.15 (C2+)
- new net C2-: IC6.10 (CS-), IC6.16 (C2-)
- new net GND: C11.1, IC6.6 (GND_1), IC6.9 (GND_2), J2.10 (Pin_10), J2.2 (Pin_2), J5.5
- new net JTAG_TCK: J2.1 (Pin_1)
- new net JTAG_TDI: J2.9 (Pin_9)
- new net JTAG_TDO: J2.3 (Pin_3)
- new net JTAG_TMS: J2.5 (Pin_5)
- new net RX_RS232: IC6.4 (R1IN), J5.2
- new net TX_RS232: IC6.5 (T1OUT), J5.3
- new net UART_RX: IC6.3 (R1OUT)
- new net UART_TX: IC6.2 (T1IN)
- new net V-: IC6.12 (V-), IC6.17 (V-)
- new net ~{RESET}: J2.6 (Pin_6)
- no-connect marks 0 -> 15

Commit message: Schematic udated
Parts:
- added C17, C18: 100n, symbol Device:C
- added C19, C20: 22p, symbol Device:C
- added R4: 120R, symbol Device:R
- added U3: MCP2515-xSO, Package_SO:TSSOP-20_4.4x6.5mm_P0.65mm, symbol Interface_CAN_LIN:MCP2515-xSO
- added U4: MCP2551-I-P, Package_DIP:DIP-8_W7.62mm, symbol Interface_CAN_LIN:MCP2551-I-P
- added Y3: 16MHz, symbol Device:Crystal
Connections:
- net +5V: now also C17.1, C18.1, U3.18 (VDD), U4.3 (VDD)
- net GND: now also C17.2, C18.2, C19.2, C20.1, U3.9 (VSS), U4.2 (VSS)
- net ~{RESET}: now also U3.17 (~{RESET})
- new net: U3.1 (TXCAN), U4.1 (TXD)
- new net: U3.2 (RXCAN), U4.4 (RXD)
- new net: R4.1, U4.7 (CANH)
- new net: R4.2, U4.6 (CANL)
- new net MISO: U3.15 (SO)
- new net MOSI: U3.14 (SI)
- new net SCK: U3.13 (SCK)
- new net XTAL1: C19.1, U3.7 (OSC2), Y3.1
- new net XTAL2: C20.2, U3.8 (OSC1), Y3.2
- new net ~{CS}: U3.16 (~{CS})
- new net ~{INT}: U3.12 (~{INT})
- no-connect marks 15 -> 21

Commit message: Finnished schematic
Parts:
- added J6: CAN, symbol Connector:Conn_01x02_Pin
- added R4: 22k, symbol Device:R
- J4: renamed from J2; value Conn_02x05_Odd_Even -> JTAG Connector
- J5: value DE9_Socket -> Til PC
- renumbered C11 to C16, C19 to C17, C20 to C18, C18 to C19, C17 to C20, IC6 to IC5, R4 to R5, Y3 to Y2
Connections:
- net GND: now also R4.2
- net CAN_TX: now reaches U3.1 (TXCAN), U4.1 (TXD)
- net CAN_RX: now reaches U3.2 (RXCAN), U4.4 (RXD)
- net CANH: now reaches R5.1, U4.7 (CANH)
- net CANH: now also J6.2 (Pin_2)
- net CANL: now reaches R5.2, U4.6 (CANL)
- net CANL: now also J6.1 (Pin_1)
- net at U4.8 (Rs): now also R4.1
- no-connect marks 21 -> 22
Other:
- note added: "Baud rate: 9600"
- note added: "CAN Interface"
- note added: "JTAG Interface"
- note added: "RS232 Interface"
- company: (none) -> Gruppe 31
- title: (none) -> Veldig pent yup yup
- moved on the sheet: C16, C17, C18, C19, C20, J4, J5, R5, U3, U4, Y2

Commit message: Liten Schematic endring
Parts:
- renumbered C19 to C16, C20 to C17, C17 to C18, C18 to C19, C16 to C20, J6 to J5, J5 to J6, R5 to R4, R4 to R5, U4 to U3, U3 to U4
Other:
- note added: "Serial interface peripherals"
Changed lines of the file:
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@@
 		)
 	)
+	(text "Serial interface peripherals"
+		(exclude_from_sim no)
+		(at 95.25 147.828 0)
+		(effects
+			(font
+				(size 5.08 5.08)
+				(thickness 1.016)
+				(bold yes)
+			)
+		)
+	)
 	(text "CAN Interface"
 		(exclude_from_sim no)
@@
 		(dnp no)
 		(fields_autoplaced yes)
-		(property "Reference" "#PWR038"
+		(property "Reference" "#PWR031"
 			(at 186.69 53.34 0)
 			(hide yes)
@@
 			(project "Byggern_Schematics"
 				(path "/26e08e78-9dbc-4948-a13f-fc9d093951ff/87d22ef8-9c9b-4de0-9f82-7ce26e0f6075"
-					(reference "#PWR038")
+					(reference "#PWR031")
 					(unit 1)
 				)
@@
 		(dnp no)
 		(fields_autoplaced yes)
-		(property "Reference" "#PWR034"
+		(property "Reference" "#PWR030"
 			(at 101.6 52.07 0)
 			(hide yes)
@@
 			(project "Byggern_Schematics"
 				(path "/26e08e78-9dbc-4948-a13f-fc9d093951ff/87d22ef8-9c9b-4de0-9f82-7ce26e0f6075"
-					(reference "#PWR034")
+					(reference "#PWR030")
 					(unit 1)
 				)
@@
 		(dnp no)
 		(fields_autoplaced yes)
-		(property "Reference" "#PWR030"
+		(property "Reference" "#PWR038"
 			(at 73.66 96.52 0)
 			(hide yes)
@@
 			(project "Byggern_Schematics"
 				(path "/26e08e78-9dbc-4948-a13f-fc9d093951ff/87d22ef8-9c9b-4de0-9f82-7ce26e0f6075"
-					(reference "#PWR030")
+					(reference "#PWR038")
 					(unit 1)
 				)
@@
 		(dnp no)
 		(fields_autoplaced yes)
-		(property "Reference" "C19"
+		(property "Reference" "C16"
 			(at 181.61 54.6099 0)
 			(show_name no)
@@
 			(project "Byggern_Schematics"
 				(path "/26e08e78-9dbc-4948-a13f-fc9d093951ff/87d22ef8-9c9b-4de0-9f82-7ce26e0f6075"
-					(reference "C19")
+					(reference "C16")
 					(unit 1)
 				)
@@
 		(dnp no)
 		(fields_autoplaced yes)
-		(property "Reference" "U3"
+		(property "Reference" "U4"
 			(at 188.8333 58.42 0)
 			(show_name no)
@@
 			(project "Byggern_Schematics"
 				(path "/26e08e78-9dbc-4948-a13f-fc9d093951ff/87d22ef8-9c9b-4de0-9f82-7ce26e0f6075"
-					(reference "U3")
+					(reference "U4")
 					(unit 1)
 				)
@@
 		(dnp no)
 		(fields_autoplaced yes)
-		(property "Reference" "#PWR033"
+		(property "Reference" "#PWR035"
 			(at 99.06 67.31 0)
 			(hide yes)
@@
 			(project "Byggern_Schematics"
 				(path "/26e08e78-9dbc-4948-a13f-fc9d093951ff/87d22ef8-9c9b-4de0-9f82-7ce26e0f6075"
-					(reference "#PWR033")
+					(reference "#PWR035")
 					(unit 1)
 				)
@@
 		(dnp no)
 		(fields_autoplaced yes)
-		(property "Reference" "#PWR035"
+		(property "Reference" "#PWR042"
 			(at 102.87 129.54 0)
 			(hide yes)
@@
 			(project "Byggern_Schematics"
 				(path "/26e08e78-9dbc-4948-a13f-fc9d093951ff/87d22ef8-9c9b-4de0-9f82-7ce26e0f6075"
-					(reference "#PWR035")
+					(reference "#PWR042")
 					(unit 1)
 				)
@@
 		(dnp no)
 		(fields_autoplaced yes)
-		(property "Reference" "C18"
+		(property "Reference" "C19"
 			(at 147.32 86.36 90)
 			(show_name no)
@@
 			(project "Byggern_Schematics"
 				(path "/26e08e78-9dbc-4948-a13f-fc9d093951ff/87d22ef8-9c9b-4de0-9f82-7ce26e0f6075"
-					(reference "C18")
+					(reference "C19")
 					(unit 1)
 				)
@@
 		(dnp no)
 		(fields_autoplaced yes)
-		(property "Reference" "#PWR040"
+		(property "Reference" "#PWR037"
 			(at 220.98 92.71 0)
 			(hide yes)
@@
 			(project "Byggern_Schematics"
 				(path "/26e08e78-9dbc-4948-a13f-fc9d093951ff/87d22ef8-9c9b-4de0-9f82-7ce26e0f6075"
-					(reference "#PWR040")
+					(reference "#PWR037")
 					(unit 1)
 				)
@@
 		(dnp no)
 		(fields_autoplaced yes)
-		(property "Reference" "J6"
+		(property "Reference" "J5"
 			(at 271.78 69.8499 0)
 			(show_name no)
@@
 			(project "Byggern_Schematics"
 				(path "/26e08e78-9dbc-4948-a13f-fc9d093951ff/87d22ef8-9c9b-4de0-9f82-7ce26e0f6075"
-					(reference "J6")
+					(reference "J5")
 					(unit 1)
 				)
@@
 		(dnp no)
 		(fields_autoplaced yes)
-		(property "Reference" "R5"
+		(property "Reference" "R4"
 			(at 252.73 69.8499 0)
 			(show_name no)
@@
 			(project "Byggern_Schematics"
 				(path "/26e08e78-9dbc-4948-a13f-fc9d093951ff/87d22ef8-9c9b-4de0-9f82-7ce26e0f6075"
-					(reference "R5")
+					(reference "R4")
 					(unit 1)
 				)
@@
 		(dnp no)
 		(fields_autoplaced yes)
-		(property "Reference" "C16"
+		(property "Reference" "C20"
 			(at 101.6 95.2499 0)
 			(show_name no)
@@
 			(project "Byggern_Schematics"
 				(path "/26e08e78-9dbc-4948-a13f-fc9d093951ff/87d22ef8-9c9b-4de0-9f82-7ce26e0f6075"
-					(reference "C16")
+					(reference "C20")
 					(unit 1)
 				)
@@
 		(dnp no)
 		(fields_autoplaced yes)
-		(property "Reference" "#PWR031"
+		(property "Reference" "#PWR043"
 			(at 76.2 137.16 0)
 			(hide yes)
@@
 			(project "Byggern_Schematics"
 				(path "/26e08e78-9dbc-4948-a13f-fc9d093951ff/87d22ef8-9c9b-4de0-9f82-7ce26e0f6075"
-					(reference "#PWR031")
+					(reference "#PWR043")
 					(unit 1)
 				)
@@
 		(dnp no)
 		(fields_autoplaced yes)
-		(property "Reference" "#PWR042"
+		(property "Reference" "#PWR032"
 			(at 234.95 53.34 0)
 			(hide yes)
@@
 			(project "Byggern_Schematics"
 				(path "/26e08e78-9dbc-4948-a13f-fc9d093951ff/87d22ef8-9c9b-4de0-9f82-7ce26e0f6075"
-					(reference "#PWR042")
+					(reference "#PWR032")
 					(unit 1)
 				)
@@
 		(dnp no)
 		(fields_autoplaced yes)
-		(property "Reference" "C17"
+		(property "Reference" "C18"
 			(at 147.32 73.66 90)
 			(show_name no)
@@
 			(project "Byggern_Schematics"
 				(path "/26e08e78-9dbc-4948-a13f-fc9d093951ff/87d22ef8-9c9b-4de0-9f82-7ce26e0f6075"
-					(reference "C17")
+					(reference "C18")
 					(unit 1)
 				)
@@
 		(dnp no)
 		(fields_autoplaced yes)
-		(property "Reference" "R4"
+		(property "Reference" "R5"
 			(at 223.52 80.0099 0)
 			(show_name no)
@@
 			(project "Byggern_Schematics"
 				(path "/26e08e78-9dbc-4948-a13f-fc9d093951ff/87d22ef8-9c9b-4de0-9f82-7ce26e0f6075"
-					(reference "R4")
+					(reference "R5")
 					(unit 1)
 				)
@@
 		(dnp no)
 		(fields_autoplaced yes)
-		(property "Reference" "#PWR039"
+		(property "Reference" "#PWR041"
 			(at 186.69 110.49 0)
 			(hide yes)
@@
 			(project "Byggern_Schematics"
 				(path "/26e08e78-9dbc-4948-a13f-fc9d093951ff/87d22ef8-9c9b-4de0-9f82-7ce26e0f6075"
-					(reference "#PWR039")
+					(reference "#PWR041")
 					(unit 1)
 				)
@@
 		(dnp no)
 		(fields_autoplaced yes)
-		(property "Reference" "#PWR032"
+		(property "Reference" "#PWR040"
 			(at 97.79 106.68 0)
 			(hide yes)
@@
 			(project "Byggern_Schematics"
 				(path "/26e08e78-9dbc-4948-a13f-fc9d093951ff/87d22ef8-9c9b-4de0-9f82-7ce26e0f6075"
-					(reference "#PWR032")
+					(reference "#PWR040")
 					(unit 1)
 				)
@@
 		(dnp no)
 		(fields_autoplaced yes)
-		(property "Reference" "U4"
+		(property "Reference" "U3"
 			(at 237.0933 58.42 0)
 			(show_name no)
@@
 			(project "Byggern_Schematics"
 				(path "/26e08e78-9dbc-4948-a13f-fc9d093951ff/87d22ef8-9c9b-4de0-9f82-7ce26e0f6075"
-					(reference "U4")
+					(reference "U3")
 					(unit 1)
 				)
@@
 		(dnp no)
 		(fields_autoplaced yes)
-		(property "Reference" "#PWR037"
+		(property "Reference" "#PWR033"
 			(at 177.8 66.04 0)
 			(hide yes)
@@
 			(project "Byggern_Schematics"
 				(path "/26e08e78-9dbc-4948-a13f-fc9d093951ff/87d22ef8-9c9b-4de0-9f82-7ce26e0f6075"
-					(reference "#PWR037")
+					(reference "#PWR033")
 					(unit 1)
 				)
@@
 		(dnp no)
 		(fields_autoplaced yes)
-		(property "Reference" "#PWR043"
+		(property "Reference" "#PWR036"
 			(at 234.95 87.63 0)
 			(hide yes)
@@
 			(project "Byggern_Schematics"
 				(path "/26e08e78-9dbc-4948-a13f-fc9d093951ff/87d22ef8-9c9b-4de0-9f82-7ce26e0f6075"
-					(reference "#PWR043")
+					(reference "#PWR036")
 					(unit 1)
 				)
@@
 		(dnp no)
 		(fields_autoplaced yes)
-		(property "Reference" "#PWR041"
+		(property "Reference" "#PWR034"
 			(at 226.06 66.04 0)
 			(hide yes)
@@
 			(project "Byggern_Schematics"
 				(path "/26e08e78-9dbc-4948-a13f-fc9d093951ff/87d22ef8-9c9b-4de0-9f82-7ce26e0f6075"
-					(reference "#PWR041")
+					(reference "#PWR034")
 					(unit 1)
 				)
@@
 		(dnp no)
 		(fields_autoplaced yes)
-		(property "Reference" "C20"
+		(property "Reference" "C17"
 			(at 229.87 54.6099 0)
 			(show_name no)
@@
 			(project "Byggern_Schematics"
 				(path "/26e08e78-9dbc-4948-a13f-fc9d093951ff/87d22ef8-9c9b-4de0-9f82-7ce26e0f6075"
-					(reference "C20")
+					(reference "C17")
 					(unit 1)
 				)
@@
 		(dnp no)
 		(fields_autoplaced yes)
-		(property "Reference" "J5"
+		(property "Reference" "J6"
 			(at 116.84 110.4899 0)
 			(show_name no)
@@
 			(project "Byggern_Schematics"
 				(path "/26e08e78-9dbc-4948-a13f-fc9d093951ff/87d22ef8-9c9b-4de0-9f82-7ce26e0f6075"
-					(reference "J5")
+					(reference "J6")
 					(unit 1)
 				)
@@
 		(dnp no)
 		(fields_autoplaced yes)
-		(property "Reference" "#PWR036"
+		(property "Reference" "#PWR039"
 			(at 140.97 102.87 0)
 			(hide yes)
@@
 			(project "Byggern_Schematics"
 				(path "/26e08e78-9dbc-4948-a13f-fc9d093951ff/87d22ef8-9c9b-4de0-9f82-7ce26e0f6075"
-					(reference "#PWR036")
+					(reference "#PWR039")
 					(unit 1)
 				)

Commit message: Små endringer til schematic
Parts:
- removed J5: CAN, symbol Connector:Conn_01x02_Pin
- renumbered C20 to C41, C18 to C42, C19 to C43, C16 to C44, C17 to C51, IC5 to IC12, J4 to J13, J6 to J14, R5 to R11, R4 to R12, U3 to U10, U4 to U9, Y2 to Y5
