File: Byggern_Schematics/ekstern_minne.kicad_sch (KiCad schematic)
At the start: 0 parts

Commit message: Byggern sjematikk for ADC done
Parts:
- added C10, C12: 100n, symbol Device:C
- added C13, C14, C15, C16, C5: 10u, symbol Device:C_Polarized
- added IC2: SN74ALS573CN, Samacsys:DIP794W53P254L2540H508Q20N, symbol Samacsys:SN74ALS573CN
- added IC3: 7164S25YG, Samacsys:7164S25YG, symbol Samacsys:7164S25YG
- added IC4: SN74HC00N, Samacsys:DIP794W53P254L1930H508Q14N, symbol Samacsys:SN74HC00N
- added IC5: MAX156BCNG+, Samacsys:DIP794W56P254L3054H457Q24N, symbol Samacsys:MAX156BCNG+
Connections:
- new net +5V: C10.1, C13.1, C14.1, C15.1, C16.1, IC2.20 (VCC), IC3.2 (A12), IC3.21 (A10), IC3.28 (VCC), IC4.14 (VCC), IC5.22 (VDD)
- new net A0: IC2.19 (1Q), IC3.10 (A0)
- new net A1: IC2.18 (2Q), IC3.9 (A1)
- new net A2: IC2.17 (3Q), IC3.8 (A2)
- new net A3: IC2.16 (4Q), IC3.7 (A3)
- new net A4: IC2.15 (5Q), IC3.6 (A4)
- new net A5: IC2.14 (6Q), IC3.5 (A5)
- new net A6: IC2.13 (7Q), IC3.4 (A6)
- new net A7: IC2.12 (8Q), IC3.3 (A7)
- new net AIN0: IC5.2 (AIN0)
- new net AIN1: IC5.1 (AIN1)
- new net AIN2: IC5.24 (AIN2)
- new net AIN3: IC5.23 (AIN3)
- new net ALE: IC2.11 (LE)
- new net CLK: IC5.9 (CLK)
- new net GND: C10.2, C12.2, C13.2, C14.2, C15.2, C16.2, C5.2, IC2.1 (~{OE}), IC2.10 (GND), IC3.14 (GND), IC3.20 (~{CS1}), IC4.7 (GND), IC5.12 (DGND), IC5.21 (AGND), IC5.4 (VSS)
- new net PA0: IC2.2 (1D), IC3.11 (I/O0), IC5.10 (D7/~{ALL})
- new net PA1: IC2.3 (2D), IC3.12 (I/O1), IC5.11 (D6/DIFF)
- new net PA2: IC2.4 (3D), IC3.13 (I/O2), IC5.13 (D5/BIP)
- new net PA3: IC2.5 (4D), IC3.15 (I/O3), IC5.14 (D4/INH)
- new net PA4: IC2.6 (5D), IC3.16 (I/O4), IC5.15 (D3/PD)
- new net PA5: IC2.7 (6D), IC3.17 (I/O5), IC5.16 (D2)
- new net PA6: IC2.8 (7D), IC3.18 (I/O6), IC5.17 (D1/A1)
- new net PA7: IC2.9 (8D), IC3.19 (I/O7), IC5.18 (D0/A0)
- new net PC0: IC3.25 (A8)
- new net PC1: IC3.24 (A9)
- new net PC2: IC3.23 (A11)
- new net PC3: IC3.26 (CS2), IC5.5 (~{CS})
- new net REF: C12.1, C5.1, IC5.19 (REFOUT), IC5.20 (REFIN)
- new net ~{BUSY}: IC5.8 (~{BUSY})
- new net ~{RD}: IC3.22 (~{OE}), IC5.6 (~{RD})
- new net ~{WR}: IC3.27 (~{WE}), IC5.7 (~{WR})
- no-connect marks 0 -> 1

Commit message: Schematic udated
Parts:
- added C9: 10u, symbol Device:C_Polarized
Connections:
- net +5V: now also C12.1, IC5.20 (REFIN), C9.1
- net GND: now also C9.2
- net REF: no longer C12.1, IC5.20 (REFIN)
- net ~{BUSY} renamed PD3
- net ~{RD} renamed PD7
- net ~{WR} renamed PD6
Other:
- moved on the sheet: C5

Commit message: Finnished schematic
Parts:
- renumbered C5 to C10, C14 to C11, C15 to C13, C9 to C14, C16 to C15, C10 to C8, C13 to C9, IC2 to IC1, IC4 to IC2, IC5 to IC4
Connections:
- net at IC2.1 (1A): now also IC2.2 (1B)
- net at IC2.10 (3B): now also IC2.3 (1Y)
- net at IC2.4 (2A): now also IC2.5 (2B)
- net at IC2.6 (2Y): now also IC2.9 (3A)
- no-connect marks 1 -> 7
Other:
- note added: "8KiB SRAM We only use 2KiB"
- note added: "ADC"
- note added: "Address decoder"
- note added: "Currently not connected or used"
- note added: "LATCH"
- note added: "Latches the address before data is sent"
- note added: "SRAM"
- company: (none) -> Gruppe 31
- title: (none) -> Veldig pent yup yup
- moved on the sheet: IC2

Commit message: Liten Schematic endring
Parts:
- renumbered C11 to C10, C13 to C11, C15 to C12, C10 to C13, C12 to C14, C14 to C15, IC3 to IC2, IC4 to IC3, IC2 to IC4
Other:
- note added: "Paralell interface peripherals"
Changed lines of the file:
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@@
 		)
 	)
+	(text "Paralell interface peripherals"
+		(exclude_from_sim no)
+		(at 144.78 21.59 0)
+		(effects
+			(font
+				(size 5.08 5.08)
+				(thickness 1.016)
+				(bold yes)
+			)
+		)
+	)
 	(text "Latches the address\nbefore data is sent"
 		(exclude_from_sim no)
@@
 		(dnp no)
 		(fields_autoplaced yes)
-		(property "Reference" "C11"
+		(property "Reference" "C10"
 			(at 217.17 51.1809 0)
 			(show_name no)
@@
 			(project "Byggern_Schematics"
 				(path "/26e08e78-9dbc-4948-a13f-fc9d093951ff/ec5cc565-6ceb-4887-a28f-4e21142ebd62"
-					(reference "C11")
+					(reference "C10")
 					(unit 1)
 				)
@@
 		(dnp no)
 		(fields_autoplaced yes)
-		(property "Reference" "#PWR019"
+		(property "Reference" "#PWR020"
 			(at 116.84 64.77 0)
 			(hide yes)
@@
 			(project "Byggern_Schematics"
 				(path "/26e08e78-9dbc-4948-a13f-fc9d093951ff/ec5cc565-6ceb-4887-a28f-4e21142ebd62"
-					(reference "#PWR019")
+					(reference "#PWR020")
 					(unit 1)
 				)
@@
 		(dnp no)
 		(fields_autoplaced yes)
-		(property "Reference" "C10"
+		(property "Reference" "C13"
 			(at 209.55 100.7109 0)
 			(show_name no)
@@
 			(project "Byggern_Schematics"
 				(path "/26e08e78-9dbc-4948-a13f-fc9d093951ff/ec5cc565-6ceb-4887-a28f-4e21142ebd62"
-					(reference "C10")
+					(reference "C13")
 					(unit 1)
 				)
@@
 		(dnp no)
 		(fields_autoplaced yes)
-		(property "Reference" "#PWR018"
+		(property "Reference" "#PWR024"
 			(at 93.98 96.52 0)
 			(hide yes)
@@
 			(project "Byggern_Schematics"
 				(path "/26e08e78-9dbc-4948-a13f-fc9d093951ff/ec5cc565-6ceb-4887-a28f-4e21142ebd62"
-					(reference "#PWR018")
+					(reference "#PWR024")
 					(unit 1)
 				)
@@
 		(dnp no)
 		(fields_autoplaced yes)
-		(property "Reference" "#PWR017"
+		(property "Reference" "#PWR029"
 			(at 90.17 184.15 0)
 			(hide yes)
@@
 			(project "Byggern_Schematics"
 				(path "/26e08e78-9dbc-4948-a13f-fc9d093951ff/ec5cc565-6ceb-4887-a28f-4e21142ebd62"
-					(reference "#PWR017")
+					(reference "#PWR029")
 					(unit 1)
 				)
@@
 		(dnp no)
 		(fields_autoplaced yes)
-		(property "Reference" "IC2"
+		(property "Reference" "IC4"
 			(at 83.82 148.59 0)
 			(show_name no)
@@
 			(project "Byggern_Schematics"
 				(path "/26e08e78-9dbc-4948-a13f-fc9d093951ff/ec5cc565-6ceb-4887-a28f-4e21142ebd62"
-					(reference "IC2")
+					(reference "IC4")
 					(unit 1)
 				)
@@
 		(dnp no)
 		(fields_autoplaced yes)
-		(property "Reference" "#PWR013"
+		(property "Reference" "#PWR021"
 			(at 50.8 71.12 0)
 			(hide yes)
@@
 			(project "Byggern_Schematics"
 				(path "/26e08e78-9dbc-4948-a13f-fc9d093951ff/ec5cc565-6ceb-4887-a28f-4e21142ebd62"
-					(reference "#PWR013")
+					(reference "#PWR021")
 					(unit 1)
 				)
@@
 		(dnp no)
 		(fields_autoplaced yes)
-		(property "Reference" "#PWR016"
+		(property "Reference" "#PWR028"
 			(at 90.17 148.59 0)
 			(hide yes)
@@
 			(project "Byggern_Schematics"
 				(path "/26e08e78-9dbc-4948-a13f-fc9d093951ff/ec5cc565-6ceb-4887-a28f-4e21142ebd62"
-					(reference "#PWR016")
+					(reference "#PWR028")
 					(unit 1)
 				)
@@
 		(dnp no)
 		(fields_autoplaced yes)
-		(property "Reference" "C14"
+		(property "Reference" "C15"
 			(at 232.41 100.7109 0)
 			(show_name no)
@@
 			(project "Byggern_Schematics"
 				(path "/26e08e78-9dbc-4948-a13f-fc9d093951ff/ec5cc565-6ceb-4887-a28f-4e21142ebd62"
-					(reference "C14")
+					(reference "C15")
 					(unit 1)
 				)
@@
 		(dnp no)
 		(fields_autoplaced yes)
-		(property "Reference" "#PWR021"
+		(property "Reference" "#PWR022"
 			(at 133.35 82.55 0)
 			(hide yes)
@@
 			(project "Byggern_Schematics"
 				(path "/26e08e78-9dbc-4948-a13f-fc9d093951ff/ec5cc565-6ceb-4887-a28f-4e21142ebd62"
-					(reference "#PWR021")
+					(reference "#PWR022")
 					(unit 1)
 				)
@@
 		(dnp no)
 		(fields_autoplaced yes)
-		(property "Reference" "#PWR020"
+		(property "Reference" "#PWR026"
 			(at 116.84 110.49 0)
 			(hide yes)
@@
 			(project "Byggern_Schematics"
 				(path "/26e08e78-9dbc-4948-a13f-fc9d093951ff/ec5cc565-6ceb-4887-a28f-4e21142ebd62"
-					(reference "#PWR020")
+					(reference "#PWR026")
 					(unit 1)
 				)
@@
 		(dnp no)
 		(fields_autoplaced yes)
-		(property "Reference" "#PWR028"
+		(property "Reference" "#PWR025"
 			(at 228.6 96.52 0)
 			(hide yes)
@@
 			(project "Byggern_Schematics"
 				(path "/26e08e78-9dbc-4948-a13f-fc9d093951ff/ec5cc565-6ceb-4887-a28f-4e21142ebd62"
-					(reference "#PWR028")
+					(reference "#PWR025")
 					(unit 1)
 				)
@@
 		(dnp no)
 		(fields_autoplaced yes)
-		(property "Reference" "#PWR029"
+		(property "Reference" "#PWR018"
 			(at 233.68 63.5 0)
 			(hide yes)
@@
 			(project "Byggern_Schematics"
 				(path "/26e08e78-9dbc-4948-a13f-fc9d093951ff/ec5cc565-6ceb-4887-a28f-4e21142ebd62"
-					(reference "#PWR029")
+					(reference "#PWR018")
 					(unit 1)
 				)
@@
 		(dnp no)
 		(fields_autoplaced yes)
-		(property "Reference" "C15"
+		(property "Reference" "C12"
 			(at 237.49 51.1809 0)
 			(show_name no)
@@
 			(project "Byggern_Schematics"
 				(path "/26e08e78-9dbc-4948-a13f-fc9d093951ff/ec5cc565-6ceb-4887-a28f-4e21142ebd62"
-					(reference "C15")
+					(reference "C12")
 					(unit 1)
 				)
@@
 		(dnp no)
 		(fields_autoplaced yes)
-		(property "Reference" "IC3"
+		(property "Reference" "IC2"
 			(at 109.22 62.23 0)
 			(show_name no)
@@
 			(project "Byggern_Schematics"
 				(path "/26e08e78-9dbc-4948-a13f-fc9d093951ff/ec5cc565-6ceb-4887-a28f-4e21142ebd62"
-					(reference "IC3")
+					(reference "IC2")
 					(unit 1)
 				)
@@
 		(dnp no)
 		(fields_autoplaced yes)
-		(property "Reference" "IC4"
+		(property "Reference" "IC3"
 			(at 172.72 62.23 0)
 			(show_name no)
@@
 			(project "Byggern_Schematics"
 				(path "/26e08e78-9dbc-4948-a13f-fc9d093951ff/ec5cc565-6ceb-4887-a28f-4e21142ebd62"
-					(reference "IC4")
+					(reference "IC3")
 					(unit 1)
 				)
@@
 		(dnp no)
 		(fields_autoplaced yes)
-		(property "Reference" "#PWR027"
+		(property "Reference" "#PWR017"
 			(at 223.52 63.5 0)
 			(hide yes)
@@
 			(project "Byggern_Schematics"
 				(path "/26e08e78-9dbc-4948-a13f-fc9d093951ff/ec5cc565-6ceb-4887-a28f-4e21142ebd62"
-					(reference "#PWR027")
+					(reference "#PWR017")
 					(unit 1)
 				)
@@
 		(dnp no)
 		(fields_autoplaced yes)
-		(property "Reference" "C12"
+		(property "Reference" "C14"
 			(at 219.71 101.5999 0)
 			(show_name no)
@@
 			(project "Byggern_Schematics"
 				(path "/26e08e78-9dbc-4948-a13f-fc9d093951ff/ec5cc565-6ceb-4887-a28f-4e21142ebd62"
-					(reference "C12")
+					(reference "C14")
 					(unit 1)
 				)
@@
 		(dnp no)
 		(fields_autoplaced yes)
-		(property "Reference" "#PWR024"
+		(property "Reference" "#PWR027"
 			(at 190.5 118.11 0)
 			(hide yes)
@@
 			(project "Byggern_Schematics"
 				(path "/26e08e78-9dbc-4948-a13f-fc9d093951ff/ec5cc565-6ceb-4887-a28f-4e21142ebd62"
-					(reference "#PWR024")
+					(reference "#PWR027")
 					(unit 1)
 				)
@@
 		(in_pos_files yes)
 		(dnp no)
-		(property "Reference" "#PWR014"
+		(property "Reference" "#PWR019"
 			(at 63.5 62.23 0)
 			(hide yes)
@@
 			(project "Byggern_Schematics"
 				(path "/26e08e78-9dbc-4948-a13f-fc9d093951ff/ec5cc565-6ceb-4887-a28f-4e21142ebd62"
-					(reference "#PWR014")
+					(reference "#PWR019")
 					(unit 1)
 				)
@@
 		(dnp no)
 		(fields_autoplaced yes)
-		(property "Reference" "C13"
+		(property "Reference" "C11"
 			(at 227.33 51.1809 0)
 			(show_name no)
@@
 			(project "Byggern_Schematics"
 				(path "/26e08e78-9dbc-4948-a13f-fc9d093951ff/ec5cc565-6ceb-4887-a28f-4e21142ebd62"
-					(reference "C13")
+					(reference "C11")
 					(unit 1)
 				)
@@
 		(dnp no)
 		(fields_autoplaced yes)
-		(property "Reference" "#PWR022"
+		(property "Reference" "#PWR013"
 			(at 184.15 50.8 0)
 			(hide yes)
@@
 			(project "Byggern_Schematics"
 				(path "/26e08e78-9dbc-4948-a13f-fc9d093951ff/ec5cc565-6ceb-4887-a28f-4e21142ebd62"
-					(reference "#PWR022")
+					(reference "#PWR013")
 					(unit 1)
 				)
@@
 		(dnp no)
 		(fields_autoplaced yes)
-		(property "Reference" "#PWR026"
+		(property "Reference" "#PWR016"
 			(at 213.36 63.5 0)
 			(hide yes)
@@
 			(project "Byggern_Schematics"
 				(path "/26e08e78-9dbc-4948-a13f-fc9d093951ff/ec5cc565-6ceb-4887-a28f-4e21142ebd62"
-					(reference "#PWR026")
+					(reference "#PWR016")
 					(unit 1)
 				)
@@
 		(dnp no)
 		(fields_autoplaced yes)
-		(property "Reference" "#PWR025"
+		(property "Reference" "#PWR015"
 			(at 203.2 63.5 0)
 			(hide yes)
@@
 			(project "Byggern_Schematics"
 				(path "/26e08e78-9dbc-4948-a13f-fc9d093951ff/ec5cc565-6ceb-4887-a28f-4e21142ebd62"
-					(reference "#PWR025")
+					(reference "#PWR015")
 					(unit 1)
 				)
@@
 		(dnp no)
 		(fields_autoplaced yes)
-		(property "Reference" "#PWR023"
+		(property "Reference" "#PWR014"
 			(at 189.23 63.5 0)
 			(hide yes)
@@
 			(project "Byggern_Schematics"
 				(path "/26e08e78-9dbc-4948-a13f-fc9d093951ff/ec5cc565-6ceb-4887-a28f-4e21142ebd62"
-					(reference "#PWR023")
+					(reference "#PWR014")
 					(unit 1)
 				)
@@
 		(dnp no)
 		(fields_autoplaced yes)
-		(property "Reference" "#PWR015"
+		(property "Reference" "#PWR023"
 			(at 63.5 97.79 0)
 			(hide yes)
@@
 			(project "Byggern_Schematics"
 				(path "/26e08e78-9dbc-4948-a13f-fc9d093951ff/ec5cc565-6ceb-4887-a28f-4e21142ebd62"
-					(reference "#PWR015")
+					(reference "#PWR023")
 					(unit 1)
 				)

Commit message: Små endringer til schematic
Parts:
- renumbered C8 to C45, C9 to C46, C13 to C47, C10 to C48, C14 to C49, C11 to C50, C15 to C52, C12 to C53, IC1 to IC11, IC4 to IC13, IC2 to IC14, IC3 to IC15
